Commit message: Add files via upload

File: arm.urdf (robot description, URDF)
Before this commit: robot servoarm, 8 links, 7 joints
Links:
- link base_link: geometry collision mesh filename=package://servoarm_description/meshes/base_cylinder.stl scale=0.0001 0.0001 0.0001; visual mesh filename=package://servoarm_description/meshes/base_cylinder.stl scale=0.0001 0.0001 0.0001
- link clawbase: geometry collision mesh filename=package://servoarm_description/meshes/clawbase.stl scale=0.001 0.001 0.001; visual mesh filename=package://servoarm_description/meshes/clawbase.stl scale=0.001 0.001 0.001
- link clawl: geometry collision mesh filename=package://servoarm_description/meshes/clawl.stl scale=0.001 0.001 0.001; visual mesh filename=package://servoarm_description/meshes/clawl.stl scale=0.001 0.001 0.001
- link clawr: geometry collision mesh filename=package://servoarm_description/meshes/clawr.stl scale=0.001 0.001 0.001; visual mesh filename=package://servoarm_description/meshes/clawr.stl scale=0.001 0.001 0.001
- link lower_arm: geometry collision mesh filename=package://servoarm_description/meshes/lower_arm.stl scale=0.001 0.001 0.001; visual mesh filename=package://servoarm_description/meshes/lower_arm.stl scale=0.001 0.001 0.001
- link platform: geometry collision mesh filename=package://servoarm_description/meshes/top_plate.stl scale=0.001 0.001 0.001; visual mesh filename=package://servoarm_description/meshes/top_plate.stl scale=0.001 0.001 0.001
- link top_arm: geometry collision mesh filename=package://servoarm_description/meshes/top_arm.stl scale=0.001 0.001 0.001; visual mesh filename=package://servoarm_description/meshes/top_arm.stl scale=0.001 0.001 0.001
- link wrist: geometry collision mesh filename=package://servoarm_description/meshes/wrist.stl scale=0.001 0.001 0.001; visual mesh filename=package://servoarm_description/meshes/wrist.stl scale=0.001 0.001 0.001
